Commit message: update joint limits

File: denso_robot_descriptions/vs060_description/vs060.urdf (robot description, URDF)
Before this commit: robot vs060, 8 links, 7 joints
Joints:
- joint joint_1: limit lower=-2.96706 upper=2.96706 effort=1 velocity=3.92699081698724 -> lower=-2.96706 upper=2.96706 effort=1 velocity=3.73064127613788
- joint joint_2: limit lower=-2.094395 upper=2.094395 effort=1 velocity=2.61799387799149 -> lower=-2.094395 upper=2.094395 effort=1 velocity=2.48709418409192
- joint joint_3: limit lower=-2.181662 upper=2.70526 effort=1 velocity=2.85832571599111 -> lower=-2.181662 upper=2.70526 effort=1 velocity=2.71540943019156
- joint joint_4: limit lower=-4.712389 upper=4.712389 effort=1 velocity=3.92699081698724 -> lower=-4.712389 upper=4.712389 effort=1 velocity=3.73064127613788
- joint joint_5: limit lower=-2.094395 upper=2.094395 effort=1 velocity=3.02168853397778 -> lower=-2.094395 upper=2.094395 effort=1 velocity=2.87060410727889
- joint joint_6: limit lower=-6.283185 upper=6.283185 effort=1 velocity=6.28318530717959 -> lower=-6.283185 upper=6.283185 effort=1 velocity=5.96902604182061

Commit message: ジョイントリミットを正しく設定。結構大事な作業かもしれない。

File: denso_robot_descriptions/vs060_description/vs060.urdf (robot description, URDF)
Before this commit: robot vs060, 8 links, 7 joints
Joints:
- joint joint_1: limit lower=-2.96706 upper=2.96706 effort=1 velocity=3.73064127613788 -> lower=-2.9 upper=2.9 effort=1 velocity=3.73064127613788
- joint joint_2: limit lower=-2.094395 upper=2.094395 effort=1 velocity=2.48709418409192 -> lower=-1.5 upper=1.5 effort=1 velocity=2.48709418409192
- joint joint_3: limit lower=-2.181662 upper=2.70526 effort=1 velocity=2.71540943019156 -> lower=-0.5 upper=2.7 effort=1 velocity=2.71540943019156
- joint joint_4: limit lower=-4.712389 upper=4.712389 effort=1 velocity=3.73064127613788 -> lower=-2.0 upper=2.0 effort=1 velocity=3.73064127613788
- joint joint_5: limit lower=-2.094395 upper=2.094395 effort=1 velocity=2.87060410727889 -> lower=-1.5 upper=1.5 effort=1 velocity=2.87060410727889
- joint joint_6: limit lower=-6.283185 upper=6.283185 effort=1 velocity=5.96902604182061 -> lower=-3.1 upper=3.1 effort=1 velocity=5.96902604182061

Commit message: 10/28 ICP test

File: denso_robot_descriptions/vs060_description/vs060.urdf (robot description, URDF)
Before this commit: robot vs060, 8 links, 7 joints
Links:
- added link zedm_base_link, mass 0.1; collision box size=0.13 0.03 0.016; visual box size=0.13 0.03 0.016
Joints:
- added joint zedm_joint: type fixed, parent J6, child zedm_base_link, origin xyz=0 0 0.033 rpy=0 0 0
